Commit message: X_Rob.urdf

File: urdf/X_Rob.urdf (robot description, URDF)
Before this commit: robot X_Rob, 6 links, 5 joints
Links:
- link Link1: geometry collision mesh filename=package://all.SLDASM/meshes/Link1.STL; visual mesh filename=package://all.SLDASM/meshes/Link1.STL
- link Link2: mass 0.393471125501396 -> 0.393471125501277; geometry collision mesh filename=package://all.SLDASM/meshes/Link2.STL; visual mesh filename=package://all.SLDASM/meshes/Link2.STL
- link Link3: geometry collision mesh filename=package://all.SLDASM/meshes/Link3.STL; visual mesh filename=package://all.SLDASM/meshes/Link3.STL
- link Link4: mass 0.184281039904593 -> 0.18428; geometry collision mesh filename=package://all.SLDASM/meshes/Link4.STL; visual mesh filename=package://all.SLDASM/meshes/Link4.STL
- link Link5: geometry collision mesh filename=package://all.SLDASM/meshes/Link5.STL; visual mesh filename=package://all.SLDASM/meshes/Link5.STL
- link base_link: geometry collision mesh filename=package://all.SLDASM/meshes/base_link.STL; visual mesh filename=package://all.SLDASM/meshes/base_link.STL
Joints:
- joint joint1: axis 0 0 0 -> 0 0 1; limit lower=-3.14 upper=3.14 effort=100 velocity=1 -> lower=-3.14 upper=3.14 effort=0 velocity=0; origin xyz=0 -0.1305 -0.0635 rpy=-3.1416 0 -3.1416 -> xyz=0 0 0 rpy=0 0 0; type fixed -> revolute
- joint joint2: axis 0 0 0 -> 0 0 1; limit lower=-3.14 upper=3.14 effort=100 velocity=1 -> lower=-3.14 upper=3.14 effort=0 velocity=0; origin xyz=0 -0.249 -0.0465 rpy=3.1416 0 0 -> xyz=0 0 0.1305 rpy=1.5708 0 1.5708; type fixed -> revolute
- joint joint3: axis 0 0 0 -> 0 0 1; limit lower=-3.14 upper=3.14 effort=100 velocity=1 -> lower=-3.14 upper=3.14 effort=0 velocity=0; origin xyz=0 0.219 -0.0465 rpy=-3.1416 0 3.1416 -> xyz=0 0.249 0 rpy=3.1416 0 1.5708; type fixed -> revolute
- joint joint4: axis 0 0 0 -> 0 0 1; limit lower=-3.14 upper=3.14 effort=100 velocity=1 -> lower=-3.14 upper=3.14 effort=0 velocity=0; origin xyz=0 0.0635 0.029 rpy=-1.5708 0 0 -> xyz=0.219 0 0 rpy=3.1416 0 0; type fixed -> revolute
- joint joint5: axis 0 0 0 -> 0 0 1; limit lower=-3.14 upper=3.14 effort=100 velocity=1 -> lower=-3.14 upper=3.14 effort=0 velocity=0; origin xyz=0 -0.0635 0.029 rpy=-1.5708 0 3.1416 -> xyz=0 0 0.0925 rpy=1.5708 0 1.5708; type fixed -> revolute
